File: hardware/board3_cavity_bowtie_2.4ghz/backscatter_tag_leggiero.kicad_pcb (KiCad board)
At the start: 2 copper layers, 50 x 45 mm, 5 parts, among them J1 PinHeader_1x03_P2.54mm, J2 SMA_EdgeMount

Commit message: Fix KiCad 9 schema compatibility, broken simulation imports, GUI CLI parsing, and documentation path leaks
Other:
- net class Default added: clearance 0.50, trace_width 0.50, via_dia 0.90, via_drill 0.40
- net class RF_50OHM added: clearance 0.50, trace_width 1.85, via_dia 0.90, via_drill 0.40
Changed lines of the file:
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@@
 	(setup
 		(stackup
-			(layer "F.SilkS"
-				(type "Top Silk Screen")
-			)
-			(layer "F.Mask"
-				(type "Top Solder Mask")
-				(thickness 0.01)
-			)
-			(layer "F.Cu"
-				(type "copper")
-				(thickness 0.035)
-			)
-			(layer "dielectric 1"
-				(type "core")
-				(thickness 1.51)
-				(material "FR4")
-				(epsilon_r 4.4)
-				(loss_tangent 0.02)
-			)
-			(layer "B.Cu"
-				(type "copper")
-				(thickness 0.035)
-			)
-			(layer "B.Mask"
-				(type "Bottom Solder Mask")
-				(thickness 0.01)
-			)
-			(layer "B.SilkS"
-				(type "Bottom Silk Screen")
-			)
+			(layer "F.SilkS" (type "Top Silk Screen"))
+			(layer "F.Mask" (type "Top Solder Mask") (thickness 0.01))
+			(layer "F.Cu" (type "copper") (thickness 0.035))
+			(layer "dielectric 1" (type "core") (thickness 1.51) (material "FR4") (epsilon_r 4.4) (loss_tangent 0.02))
+			(layer "B.Cu" (type "copper") (thickness 0.035))
+			(layer "B.Mask" (type "Bottom Solder Mask") (thickness 0.01))
+			(layer "B.SilkS" (type "Bottom Silk Screen"))
 			(copper_finish "None")
 			(dielectric_constraints yes)
@@
 		(pad_to_mask_clearance 0)
 		(allow_soldermask_bridges_in_footprints yes)
-		(tenting
-			(front yes)
-			(back yes)
-		)
-		(covering
-			(front no)
-			(back no)
-		)
-		(plugging
-			(front no)
-			(back no)
-		)
-		(capping no)
-		(filling no)
 		(pcbplotparams
 			(layerselection 0x00000000_00000000_00000000_02000005)
-			(plot_on_all_layers_selection 0x00000000_00000000_00000000_00000000)
 			(disableapertmacros no)
 			(usegerberextensions no)
@@
 			(usegerberadvancedattributes yes)
 			(creategerberjobfile yes)
-			(dashed_line_dash_ratio 12)
-			(dashed_line_gap_ratio 3)
-			(svgprecision 4)
-			(plotframeref no)
 			(mode 1)
 			(useauxorigin no)
-			(pdf_front_fp_property_popups yes)
-			(pdf_back_fp_property_popups yes)
-			(pdf_metadata yes)
-			(pdf_single_document no)
 			(dxfpolygonmode yes)
 			(dxfimperialunits no)
 			(dxfusepcbnewfont yes)
-			(psnegative no)
-			(psa4output no)
-			(plot_black_and_white yes)
-			(sketchpadsonfab no)
-			(plotpadnumbers no)
-			(hidednponfab no)
-			(sketchdnponfab yes)
-			(crossoutdnponfab yes)
-			(subtractmaskfromsilk no)
 			(outputformat 1)
-			(mirror no)
-			(drillshape 1)
-			(scaleselection 1)
 			(outputdirectory "gerbers")
 		)
+	)
+	(net 0 "")
+	(net 1 "GND")
+	(net 2 "/FEED")
+	(net 3 "/SMA_FEED")
+	(net 4 "/TERM_50R")
+	(net_class "Default"
+		"Standard netclass with >= 0.40 mm CNC isolation clearance"
+		(clearance 0.50)
+		(trace_width 0.50)
+		(via_dia 0.90)
+		(via_drill 0.40)
+		(uvia_dia 0.50)
+		(uvia_drill 0.25)
+	)
+	(net_class "RF_50OHM"
+		"50 Ohm Grounded Coplanar Waveguide (CPWG) with W=1.85mm, G=0.50mm"
+		(clearance 0.50)
+		(trace_width 1.85)
+		(via_dia 0.90)
+		(via_drill 0.40)
+		(uvia_dia 0.50)
+		(uvia_drill 0.25)
+		(add_net "/FEED")
+		(add_net "/SMA_FEED")
 	)
 	(property "ProjectEngineer" "M2 Worker Agent")
@@
 		(attr exclude_from_pos_files exclude_from_bom)
 		(net_tie_pad_groups "1,2")
-		(duplicate_pad_numbers_are_jumpers no)
 		(fp_poly
 			(pts
@@
 			(size 1 1)
 			(layers "F.Cu")
-			(net "/FEED")
+			(net 2 "/FEED")
 		)
 		(pad "2" smd rect
@@
 			(size 1.5 1)
 			(layers "F.Cu" "F.Mask")
-			(net "GND")
+			(net 1 "GND")
 			(zone_connect 2)
 		)
-		(embedded_fonts no)
 	)
 	(footprint "Connector_Coaxial:SMA_Samtec_SMA-J-P-H-ST-EM1_EdgeMount"
@@
 		)
 		(attr smd)
-		(duplicate_pad_numbers_are_jumpers no)
 		(pad "1" smd roundrect
 			(at 0 0)
@@
 			(layers "F.Cu" "F.Mask")
 			(roundrect_rratio 0.2)
-			(net "/SMA_FEED")
+			(net 3 "/SMA_FEED")
 		)
 		(pad "2" smd roundrect
@@
 			(layers "F.Cu" "F.Mask")
 			(roundrect_rratio 0.2)
-			(net "GND")
+			(net 1 "GND")
 			(zone_connect 2)
 		)
@@
 			(layers "F.Cu" "F.Mask")
 			(roundrect_rratio 0.2)
-			(net "GND")
+			(net 1 "GND")
 			(zone_connect 2)
 		)
-		(embedded_fonts no)
 	)
 	(footprint "Connector_PinHeader_2.54mm:PinHeader_1x03_P2.54mm_Vertical"
@@
 		)
 		(attr through_hole)
-		(duplicate_pad_numbers_are_jumpers no)
 		(pad "1" thru_hole rect
 			(at -2.54 0)
@@
 			(layers "*.Cu" "*.Mask")
 			(remove_unused_layers no)
-			(net "/TERM_50R")
+			(net 4 "/TERM_50R")
 		)
 		(pad "2" thru_hole circle
@@
 			(layers "*.Cu" "*.Mask")
 			(remove_unused_layers no)
-			(net "/FEED")
+			(net 2 "/FEED")
 		)
 		(pad "3" thru_hole circle
@@
 			(layers "*.Cu" "*.Mask")
 			(remove_unused_layers no)
-			(net "GND")
+			(net 1 "GND")
 			(zone_connect 2)
 		)
-		(embedded_fonts no)
 	)
 	(footprint "Resistor_SMD:R_0805_2012Metric"
@@
 		)
 		(attr smd)
-		(duplicate_pad_numbers_are_jumpers no)
 		(pad "1" smd roundrect
 			(at 0 -0.9125)
@@
 			(layers "F.Cu" "F.Mask")
 			(roundrect_rratio 0.25)
-			(net "GND")
+			(net 1 "GND")
 			(zone_connect 2)
 		)
@@
 			(layers "F.Cu" "F.Mask")
 			(roundrect_rratio 0.25)
-			(net "/TERM_50R")
-		)
-		(embedded_fonts no)
+			(net 4 "/TERM_50R")
+		)
 	)
 	(footprint "Resistor_SMD:R_0805_2012Metric"
@@
 		)
 		(attr smd)
-		(duplicate_pad_numbers_are_jumpers no)
 		(pad "1" smd roundrect
 			(at 0 -0.9125)
@@
 			(layers "F.Cu" "F.Mask")
 			(roundrect_rratio 0.25)
-			(net "/FEED")
+			(net 2 "/FEED")
 		)
 		(pad "2" smd roundrect
@@
 			(layers "F.Cu" "F.Mask")
 			(roundrect_rratio 0.25)
-			(net "/SMA_FEED")
-		)
-		(embedded_fonts no)
+			(net 3 "/SMA_FEED")
+		)
 	)
 	(gr_line
@@
 		(width 1.85)
 		(layer "F.Cu")
-		(net "/FEED")
+		(net 2)
 	)
 	(segment
@@
 		(width 1.85)
 		(layer "F.Cu")
-		(net "/FEED")
+		(net 2)
 	)
 	(segment
@@
 		(width 1.85)
 		(layer "F.Cu")
-		(net "/SMA_FEED")
+		(net 3)
 	)
 	(segment
@@
 		(width 0.5)
 		(layer "F.Cu")
-		(net "/TERM_50R")
-	)
-	(zone
-		(net "GND")
+		(net 4)
+	)
+	(zone (net 1) (net_name "GND")
 		(layer "F.Cu")
 		(hatch edge 0.5)
@@
 		)
 	)
-	(embedded_fonts no)
 )
